File: PCB, Schematic and Components/PCB, Schematic and Components.kicad_sch (KiCad schematic)
At the start: 7 parts, among them J1 motor, J2 Conn_01x05_Socket, Q1 IRF3205, Q2 BC547, U1 L7805

Commit message: Creation of menu and casing update
Parts:
- added C1: 330nf, Capacitor_THT:C_Disc_D3.8mm_W2.6mm_P2.50mm, symbol Device:C
- added C2, C3: 100nf, Capacitor_THT:C_Disc_D3.8mm_W2.6mm_P2.50mm, symbol Device:C
- added D1: LED, LED_THT:LED_D5.0mm, symbol Device:LED
- added J3: Measure_encoder, Connector_Hirose:Hirose_DF13-05P-1.25DSA_1x05_P1.25mm_Vertical, symbol Connector:Conn_01x05_Socket
- added J4: User_encoder, Connector_Hirose:Hirose_DF13-05P-1.25DSA_1x05_P1.25mm_Vertical, symbol Connector:Conn_01x05_Socket
- added J5: motor_led, Connector_AMASS:AMASS_XT30U-F_1x02_P5.0mm_Vertical, symbol Connector:Conn_01x02_Socket
- added R3, R4: 1k, Resistor_THT:R_Axial_DIN0207_L6.3mm_D2.5mm_P10.16mm_Horizontal, symbol Device:R
- added TP1, TP2, TP3, TP4: TestPoint, Connector_Pin:Pin_D0.7mm_L6.5mm_W1.8mm_FlatFork, symbol Connector:TestPoint
- added U2: (no value), Package_DFN_QFN:QFN-80-1EP_10x10mm_P0.4mm_EP3.4x3.4mm, symbol library:RP2350b-WeAct-Studio
- J2: value Conn_01x05_Socket -> Display
Connections:
- net +12V: now also J1.1 (Pin_1), C1.1, C3.1; no longer Q1.2 (D)
- net GND: now also Q1.3 (S), C1.2, C2.2, J3.1 (Pin_1), J4.1 (Pin_1), J5.1 (Pin_1), R3.2, TP2.1, U2.G; no longer J1.2 (Pin_2)
- net at J2.1 (Pin_1), U1.3 (OUT): now also C2.1, D1.2 (A), J3.2 (Pin_2), J4.2 (Pin_2), TP1.1, U2.VBUS
- net at Q1.1 (G), Q2.1 (C), R1.2: now also R4.1, TP4.1
- net at R2.1: now also TP3.1, U2.10
- net at J2.3 (Pin_3): now also U2.19
- net at J2.4 (Pin_4): now also U2.17
- net at J2.5 (Pin_5): now also U2.18
- new net: J3.3 (Pin_3), U2.4
- new net: J3.4 (Pin_4), U2.3
- new net: J3.5 (Pin_5), U2.2
- new net: J4.5 (Pin_5), U2.6
- new net: J4.4 (Pin_4), U2.7
- new net: J4.3 (Pin_3), U2.8
- new net: J5.2 (Pin_2), R4.2
- new net: D1.1 (K), R3.1
- new net: C3.2, J1.2 (Pin_2), Q1.2 (D)
Other:
- moved on the sheet: Q1, Q2, R2, U1
